Commit message: addtion modify

File: addition/haique_description/urdf/haique.xacro (robot description, xacro)
@@ -78,4 +78,15 @@
         <axis xyz="0 1 0" />
     </joint>
+    <!-- zuoqingzhuan_joint Transmission -->
+    <transmission name="$(arg namespace)/zuoqingzhuan_tran">
+        <type>transmission_interface/SimpleTransmission</type>
+        <joint name="$(arg namespace)/zuoqingzhuan_joint">
+            <hardwareInterface>hardware_interface/EffortJointInterface</hardwareInterface>
+        </joint>
+        <actuator name="$(arg namespace)/zuoqingzhuan_motor">
+            <hardwareInterface>hardware_interface/EffortJointInterface</hardwareInterface>
+            <mechanicalReduction>1</mechanicalReduction>
+        </actuator>
+    </transmission>
     <link name="$(arg namespace)/you_link">
         <inertial>
@@ -110,15 +121,26 @@
         <child link="$(arg namespace)/you_link" />
     </joint>
+    <!-- youqingzhuan_joint Transmission -->
+    <transmission name="$(arg namespace)/youqingzhuan_tran">
+        <type>transmission_interface/SimpleTransmission</type>
+        <joint name="$(arg namespace)/youqingzhuan_joint">
+            <hardwareInterface>hardware_interface/EffortJointInterface</hardwareInterface>
+        </joint>
+        <actuator name="$(arg namespace)/youqingzhuan_motor">
+            <hardwareInterface>hardware_interface/EffortJointInterface</hardwareInterface>
+            <mechanicalReduction>1</mechanicalReduction>
+        </actuator>
+    </transmission>
      <!-- Default joint state publisher -->
     <gazebo>
-    <plugin name="uuv_joint_state_publisher" filename="libuuv_joint_state_publisher.so">
-        <robotNamespace>$(arg namespace)</robotNamespace>
-        <updateRate>50</updateRate>
-    </plugin>
+        <plugin name="uuv_joint_state_publisher" filename="libuuv_joint_state_publisher.so">
+            <robotNamespace>$(arg namespace)</robotNamespace>
+            <updateRate>50</updateRate>
+        </plugin>
     </gazebo>
     <gazebo>
         <plugin name="gazebo_ros_control" filename="libgazebo_ros_control.so">
             <robotNamespace>/$(arg namespace)</robotNamespace>
-            <robotParam>/$(arg namespace)</robotParam>
+            <robotParam>/$(arg namespace)/haique</robotParam>
         </plugin>
     </gazebo>

Commit message: only attitude control, add eso

File: addition/haique_description/urdf/haique.xacro (robot description, xacro)
@@ -76,5 +76,6 @@
         <parent link="$(arg namespace)/haique_link" />
         <child link="$(arg namespace)/zuo_link" />
-        <axis xyz="0 1 0" />
+        <axis xyz="0 -1 0" />
+        <limit effort="4" velocity="300" />
     </joint>
     <!-- zuoqingzhuan_joint Transmission -->
@@ -120,4 +121,5 @@
         <parent link="$(arg namespace)/haique_link" />
         <child link="$(arg namespace)/you_link" />
+        <limit effort="4" velocity="300" />
     </joint>
     <!-- youqingzhuan_joint Transmission -->

File: addition/haique_description/urdf/haique_trans.urdf (robot description, URDF)
Before this commit: robot haique, 12 links, 11 joints
Joints:
- joint haique/youqingzhuan_joint: limit (none) -> effort=4 velocity=300
- joint haique/zuoqingzhuan_joint: axis 0 1 0 -> 0 -1 0; limit (none) -> effort=4 velocity=300
